File: Radio/Radio.sch (KiCad schematic (older format))
At the start: 12 parts, among them J1 USB_B_Micro, U1 FT231XS, U2 XB3

Commit message: Added proper xbee footprint, did initial layout
Parts:
- added J2: Conn_Coaxial, Connector_Coaxial:SMA_Amphenol_132289_EdgeMount, symbol Connector:Conn_Coaxial
- U2: footprint XCVR_XB3-24Z8CM-J:XCVR_XB3-24Z8CM-J -> Radio:XB3-24Z8RM-J
Connections:
- wire segments 33 -> 36
Changed lines of the file:
@@
 EESchema Schematic File Version 4
+LIBS:Radio-cache
 EELAYER 29 0
 EELAYER END
@@
 Wire Wire Line
 	1300 2950 1350 2950
-Connection ~ 5450 4150
+$Comp
+L Connector:Conn_Coaxial J2
+U 1 1 5E0856CD
+P 6700 2850
+F 0 "J2" H 6800 2825 50  0000 L CNN
+F 1 "Conn_Coaxial" H 6800 2734 50  0000 L CNN
+F 2 "Connector_Coaxial:SMA_Amphenol_132289_EdgeMount" H 6700 2850 50  0001 C CNN
+F 3 " ~" H 6700 2850 50  0001 C CNN
+	1    6700 2850
+	1    0    0    -1
+$EndComp
+Wire Wire Line
+	6150 2850 6500 2850
 $Comp
 L XB3:XB3 U2
@@
 F 0 "U2" H 5450 4031 50  0000 C CNN
 F 1 "XB3" H 5450 3940 50  0000 C CNN
-F 2 "XCVR_XB3-24Z8CM-J:XCVR_XB3-24Z8CM-J" H 5450 3250 50  0001 C CNN
+F 2 "Radio:XB3-24Z8RM-J" H 5450 3250 50  0001 C CNN
 F 3 "" H 5450 3250 50  0001 C CNN
 	1    5450 3250
@@
 $EndComp
 Wire Wire Line
-	5250 4150 5350 4150
-Wire Wire Line
-	5450 4150 5550 4150
-Connection ~ 5350 4150
-Wire Wire Line
-	5350 4150 5450 4150
-Connection ~ 5550 4150
-Wire Wire Line
-	5550 4150 5650 4150
+	5200 4150 5300 4150
+Connection ~ 5300 4150
+Wire Wire Line
+	5300 4150 5400 4150
+Connection ~ 5400 4150
+Wire Wire Line
+	5400 4150 5450 4150
+Connection ~ 5500 4150
+Wire Wire Line
+	5500 4150 5600 4150
+Connection ~ 5600 4150
+Wire Wire Line
+	5600 4150 5700 4150
+Connection ~ 5450 4150
+Wire Wire Line
+	5450 4150 5500 4150
+$Comp
+L power:GND #PWR?
+U 1 1 5E0938CD
+P 6700 3050
+F 0 "#PWR?" H 6700 2800 50  0001 C CNN
+F 1 "GND" H 6705 2877 50  0000 C CNN
+F 2 "" H 6700 3050 50  0001 C CNN
+F 3 "" H 6700 3050 50  0001 C CNN
+	1    6700 3050
+	1    0    0    -1
+$EndComp
 $EndSCHEMATC

Commit message: Revised layout significantly
Parts:
- added C?: 1uF, Capacitor_SMD:C_0805_2012Metric_Pad1.15x1.40mm_HandSolder, symbol Device:C
- added C?: 8.2pf, Capacitor_SMD:C_0805_2012Metric_Pad1.15x1.40mm_HandSolder, symbol Device:C
Connections:
- net +3V3: now also C?.1, C?.1
- net GND: now also C?.2, C?.2
Other:
- moved on the sheet: C6
Changed lines of the file:
@@
 L Device:C C6
 U 1 1 5DE006FC
-P 4400 3450
-F 0 "C6" H 4515 3496 50  0000 L CNN
-F 1 "10uF" H 4515 3405 50  0000 L CNN
-F 2 "Capacitor_SMD:C_0805_2012Metric_Pad1.15x1.40mm_HandSolder" H 4438 3300 50  0001 C CNN
-F 3 "~" H 4400 3450 50  0001 C CNN
-	1    4400 3450
+P 4400 3750
+F 0 "C6" H 4515 3796 50  0000 L CNN
+F 1 "10uF" H 4515 3705 50  0000 L CNN
+F 2 "Capacitor_SMD:C_0805_2012Metric_Pad1.15x1.40mm_HandSolder" H 4438 3600 50  0001 C CNN
+F 3 "~" H 4400 3750 50  0001 C CNN
+	1    4400 3750
 	1    0    0    -1
 $EndComp
@@
 L power:+3V3 #PWR0113
 U 1 1 5DE02652
-P 4400 3300
-F 0 "#PWR0113" H 4400 3150 50  0001 C CNN
-F 1 "+3V3" H 4415 3473 50  0000 C CNN
-F 2 "" H 4400 3300 50  0001 C CNN
-F 3 "" H 4400 3300 50  0001 C CNN
-	1    4400 3300
+P 4200 3600
+F 0 "#PWR0113" H 4200 3450 50  0001 C CNN
+F 1 "+3V3" H 4215 3773 50  0000 C CNN
+F 2 "" H 4200 3600 50  0001 C CNN
+F 3 "" H 4200 3600 50  0001 C CNN
+	1    4200 3600
 	1    0    0    -1
 $EndComp
@@
 L power:GND #PWR0114
 U 1 1 5DE02B86
-P 4400 3600
-F 0 "#PWR0114" H 4400 3350 50  0001 C CNN
-F 1 "GND" H 4405 3427 50  0000 C CNN
-F 2 "" H 4400 3600 50  0001 C CNN
-F 3 "" H 4400 3600 50  0001 C CNN
-	1    4400 3600
+P 4200 3900
+F 0 "#PWR0114" H 4200 3650 50  0001 C CNN
+F 1 "GND" H 4205 3727 50  0000 C CNN
+F 2 "" H 4200 3900 50  0001 C CNN
+F 3 "" H 4200 3900 50  0001 C CNN
+	1    4200 3900
 	1    0    0    -1
 $EndComp
@@
 	5450 4150 5500 4150
 $Comp
-L power:GND #PWR?
+L power:GND #PWR0115
 U 1 1 5E0938CD
 P 6700 3050
-F 0 "#PWR?" H 6700 2800 50  0001 C CNN
+F 0 "#PWR0115" H 6700 2800 50  0001 C CNN
 F 1 "GND" H 6705 2877 50  0000 C CNN
 F 2 "" H 6700 3050 50  0001 C CNN
@@
 	1    0    0    -1
 $EndComp
+$Comp
+L Device:C C?
+U 1 1 5E0B5CE0
+P 4200 3750
+F 0 "C?" H 4100 3850 50  0000 L CNN
+F 1 "1uF" H 4200 3650 50  0000 L CNN
+F 2 "Capacitor_SMD:C_0805_2012Metric_Pad1.15x1.40mm_HandSolder" H 4238 3600 50  0001 C CNN
+F 3 "~" H 4200 3750 50  0001 C CNN
+	1    4200 3750
+	1    0    0    -1
+$EndComp
+$Comp
+L Device:C C?
+U 1 1 5E0B6937
+P 4000 3750
+F 0 "C?" H 3700 3800 50  0000 L CNN
+F 1 "8.2pf" H 3700 3700 50  0000 L CNN
+F 2 "Capacitor_SMD:C_0805_2012Metric_Pad1.15x1.40mm_HandSolder" H 4038 3600 50  0001 C CNN
+F 3 "~" H 4000 3750 50  0001 C CNN
+	1    4000 3750
+	1    0    0    -1
+$EndComp
+Wire Wire Line
+	4000 3600 4200 3600
+Connection ~ 4200 3600
+Wire Wire Line
+	4200 3600 4400 3600
+Wire Wire Line
+	4000 3900 4200 3900
+Connection ~ 4200 3900
+Wire Wire Line
+	4200 3900 4400 3900
 $EndSCHEMATC

Commit message: Shrank RP-SMA footprint
Parts:
- J2: footprint Connector_Coaxial:SMA_Amphenol_132289_EdgeMount -> Connector_Coaxial:SMA_Samtec_SMA-J-P-H-ST-EM1_EdgeMount
- gave numbers to parts that had none: 2
Changed lines of the file:
@@
 F 0 "J2" H 6800 2825 50  0000 L CNN
 F 1 "Conn_Coaxial" H 6800 2734 50  0000 L CNN
-F 2 "Connector_Coaxial:SMA_Amphenol_132289_EdgeMount" H 6700 2850 50  0001 C CNN
+F 2 "Connector_Coaxial:SMA_Samtec_SMA-J-P-H-ST-EM1_EdgeMount" H 6700 2850 50  0001 C CNN
 F 3 " ~" H 6700 2850 50  0001 C CNN
 	1    6700 2850
@@
 $EndComp
 $Comp
-L Device:C C?
+L Device:C C8
 U 1 1 5E0B5CE0
 P 4200 3750
-F 0 "C?" H 4100 3850 50  0000 L CNN
+F 0 "C8" H 4100 3850 50  0000 L CNN
 F 1 "1uF" H 4200 3650 50  0000 L CNN
 F 2 "Capacitor_SMD:C_0805_2012Metric_Pad1.15x1.40mm_HandSolder" H 4238 3600 50  0001 C CNN
@@
 $EndComp
 $Comp
-L Device:C C?
+L Device:C C7
 U 1 1 5E0B6937
 P 4000 3750
-F 0 "C?" H 3700 3800 50  0000 L CNN
+F 0 "C7" H 3700 3800 50  0000 L CNN
 F 1 "8.2pf" H 3700 3700 50  0000 L CNN
 F 2 "Capacitor_SMD:C_0805_2012Metric_Pad1.15x1.40mm_HandSolder" H 4038 3600 50  0001 C CNN

Commit message: Add LCSC part numbers
Parts:
- C1, C5: LCSC (none) -> C49678
- C2, C4: LCSC (none) -> C14857
- C3: LCSC (none) -> C1779
- C6: LCSC (none) -> C15525
- C7: LCSC (none) -> C170111
- C8: LCSC (none) -> C28323
- R1, R2: LCSC (none) -> C17594
- U1: LCSC (none) -> C89607
Changed lines of the file:
@@
 F 2 "Package_SO:SSOP-20_3.9x8.7mm_P0.635mm" H 4250 1400 50  0001 C CNN
 F 3 "http://www.ftdichip.com/Products/ICs/FT231X.html" H 3650 2350 50  0001 C CNN
+F 4 "C89607" H 3650 2350 50  0001 C CNN "LCSC"
 	1    3650 2350
 	1    0    0    1
@@
 F 2 "Resistor_SMD:R_0805_2012Metric_Pad1.15x1.40mm_HandSolder" V 2640 2640 50  0001 C CNN
 F 3 "~" H 2600 2650 50  0001 C CNN
+F 4 "C17594" V 2600 2650 50  0001 C CNN "LCSC"
 	1    2600 2650
 	0    1    1    0
@@
 F 2 "Resistor_SMD:R_0805_2012Metric_Pad1.15x1.40mm_HandSolder" V 2340 2540 50  0001 C CNN
 F 3 "~" H 2300 2550 50  0001 C CNN
+F 4 "C17594" V 2300 2550 50  0001 C CNN "LCSC"
 	1    2300 2550
 	0    1    1    0
@@
 F 2 "Capacitor_SMD:C_0805_2012Metric_Pad1.15x1.40mm_HandSolder" H 2038 2600 50  0001 C CNN
 F 3 "~" H 2000 2750 50  0001 C CNN
+F 4 "C14857" H 2000 2750 50  0001 C CNN "LCSC"
 	1    2000 2750
 	1    0    0    -1
@@
 F 2 "Capacitor_SMD:C_0805_2012Metric_Pad1.15x1.40mm_HandSolder" H 2438 2700 50  0001 C CNN
 F 3 "~" H 2400 2850 50  0001 C CNN
+F 4 "C14857" H 2400 2850 50  0001 C CNN "LCSC"
 	1    2400 2850
 	1    0    0    -1
@@
 F 2 "Capacitor_SMD:C_0805_2012Metric_Pad1.15x1.40mm_HandSolder" H 1938 1950 50  0001 C CNN
 F 3 "~" H 1900 2100 50  0001 C CNN
+F 4 "C49678" H 1900 2100 50  0001 C CNN "LCSC"
 	1    1900 2100
 	1    0    0    -1
@@
 F 2 "Capacitor_SMD:C_0805_2012Metric_Pad1.15x1.40mm_HandSolder" H 2388 1950 50  0001 C CNN
 F 3 "~" H 2350 2100 50  0001 C CNN
+F 4 "C1779" H 2350 2100 50  0001 C CNN "LCSC"
 	1    2350 2100
 	1    0    0    -1
@@
 F 2 "Capacitor_SMD:C_0805_2012Metric_Pad1.15x1.40mm_HandSolder" H 2838 2950 50  0001 C CNN
 F 3 "~" H 2800 3100 50  0001 C CNN
+F 4 "C49678" H 2800 3100 50  0001 C CNN "LCSC"
 	1    2800 3100
 	1    0    0    -1
@@
 F 2 "Capacitor_SMD:C_0805_2012Metric_Pad1.15x1.40mm_HandSolder" H 4438 3600 50  0001 C CNN
 F 3 "~" H 4400 3750 50  0001 C CNN
+F 4 "C15525" H 4400 3750 50  0001 C CNN "LCSC"
 	1    4400 3750
 	1    0    0    -1
@@
 F 2 "Capacitor_SMD:C_0805_2012Metric_Pad1.15x1.40mm_HandSolder" H 4238 3600 50  0001 C CNN
 F 3 "~" H 4200 3750 50  0001 C CNN
+F 4 "C28323" H 4200 3750 50  0001 C CNN "LCSC"
 	1    4200 3750
 	1    0    0    -1
@@
 F 2 "Capacitor_SMD:C_0805_2012Metric_Pad1.15x1.40mm_HandSolder" H 4038 3600 50  0001 C CNN
 F 3 "~" H 4000 3750 50  0001 C CNN
+F 4 "C170111" H 4000 3750 50  0001 C CNN "LCSC"
 	1    4000 3750
 	1    0    0    -1
